File: Hardware/Simple/simple002/EAGLE/simple002.brd (EAGLE design)
At the start: 54.3 x 81.3 mm, 31 parts

Commit message: #8 hardware simple002 correct fan6 PWM to support Teensy 3.2, 3.5, 3.6, 4.0
Parts:
- removed JP1: JP1, jumper:JP1
- added SH1: SHORTT5, shorts:SHORT_TOP-50
Connections:
- net AREF: now also SH1.2; no longer JP1.2
- net HDR_PWM6: now also TEENSY.22/A8; no longer TEENSY.16/A2
- net V3.3: now also SH1.1; no longer JP1.1
Routing:
- net HDR_PWM6: track 48.6 -> 64.9 mm
- net AREF: track 69.4 -> 63.2 mm
- net V3.3: track 38.2 -> 42.6 mm
Other:
- board text removed: "(NC for Teensy 4.0)"
Changed lines of the file:
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@@
 <text x="50.8" y="76.2" size="1.016" layer="25" align="top-right">SIMPLE 002</text>
 <text x="23.241" y="57.785" size="0.762" layer="25">(Teensy 3.x, 4.0)</text>
-<text x="31.242" y="40.005" size="0.635" layer="25" rot="R90">(NC for Teensy 4.0)</text>
 </plain>
 <attributes>
@@
 <attribute name="VALUE" x="40.386" y="72.644" size="1.27" layer="27" ratio="10"/>
 </element>
-<element name="JP1" library="jumper" library_urn="urn:adsk.eagle:library:252" package="JP1" package3d_urn="urn:adsk.eagle:package:15455/1" value="JP1" x="27.94" y="43.18" smashed="yes" rot="R270">
-<attribute name="DESC" value="Break Away Headers - Straight" x="27.94" y="43.18" size="1.778" layer="27" rot="R270" display="off"/>
-<attribute name="DIGIKEY_PART_NUMBER" value="PRT-00116" x="27.94" y="43.18" size="1.778" layer="27" rot="R270" display="off"/>
-<attribute name="MANUFACTURER" value="SparkFun Electronics" x="27.94" y="43.18" size="1.778" layer="27" rot="R270" display="off"/>
-<attribute name="MANUFACTURER_PART_NUMBER" value="PRT-00116" x="27.94" y="43.18" size="1.778" layer="27" rot="R270" display="off"/>
-<attribute name="NAME" x="25.4" y="44.831" size="1.27" layer="25" ratio="10"/>
-<attribute name="POPULARITY" value="61" x="27.94" y="43.18" size="1.778" layer="27" rot="R270" display="off"/>
-<attribute name="VALUE" x="25.4" y="40.259" size="1.27" layer="27" ratio="10"/>
-</element>
 <element name="C1" library="capacitor-wima" library_urn="urn:adsk.eagle:library:116" package="C2.5-3" package3d_urn="urn:adsk.eagle:package:5436/1" value="0.1uF" x="48.006" y="69.85" smashed="yes" rot="R270">
 <attribute name="DESC" value="CAP CER 0.1UF 100V Z5U RADIAL" x="48.006" y="69.85" size="1.778" layer="27" rot="R270" display="off"/>
@@
 <attribute name="NAME" x="41.529" y="59.69" size="1.27" layer="25" rot="R270"/>
 <attribute name="VALUE" x="38.862" y="60.325" size="1.27" layer="27" rot="R270"/>
+</element>
+<element name="SH1" library="shorts" package="SHORT_TOP-50" value="SHORTT5" x="38.862" y="51.181" smashed="yes" rot="R90">
+<attribute name="BOM" value="no" x="38.862" y="51.181" size="1.778" layer="27" rot="R90" display="off"/>
+<attribute name="NAME" x="40.894" y="49.911" size="1.27" layer="25" ratio="16" rot="R90"/>
 </element>
 </elements>
@@
 <vertex x="36.576" y="27.686"/>
 <vertex x="34.036" y="27.686"/>
-<vertex x="34.036" y="30.734"/>
-<vertex x="36.576" y="30.734"/>
-<vertex x="36.576" y="37.846"/>
-<vertex x="34.036" y="37.846"/>
+<vertex x="34.036" y="48.514"/>
+<vertex x="36.576" y="48.514"/>
+<vertex x="36.576" y="50.546"/>
+<vertex x="34.036" y="50.546"/>
 <vertex x="34.036" y="58.674"/>
 <vertex x="44.069" y="58.674"/>
@@
 <vertex x="36.576" y="27.686"/>
 <vertex x="34.036" y="27.686"/>
-<vertex x="34.036" y="30.734"/>
-<vertex x="36.576" y="30.734"/>
-<vertex x="36.576" y="37.846"/>
-<vertex x="34.036" y="37.846"/>
+<vertex x="34.036" y="48.514"/>
+<vertex x="36.576" y="48.514"/>
+<vertex x="36.576" y="50.546"/>
+<vertex x="34.036" y="50.546"/>
 <vertex x="34.036" y="58.674"/>
 <vertex x="44.069" y="58.674"/>
@@
 <vertex x="43.815" y="58.166"/>
 <vertex x="34.544" y="58.166"/>
-<vertex x="34.544" y="38.354"/>
-<vertex x="37.211" y="38.354"/>
-<vertex x="37.211" y="30.226"/>
-<vertex x="34.544" y="30.226"/>
+<vertex x="34.544" y="51.054"/>
+<vertex x="37.211" y="51.054"/>
+<vertex x="37.211" y="48.006"/>
+<vertex x="34.544" y="48.006"/>
 <vertex x="34.544" y="28.194"/>
 <vertex x="37.211" y="28.194"/>
@@
 <vertex x="43.815" y="58.166"/>
 <vertex x="34.544" y="58.166"/>
-<vertex x="34.544" y="38.354"/>
-<vertex x="37.211" y="38.354"/>
-<vertex x="37.211" y="30.226"/>
-<vertex x="34.544" y="30.226"/>
+<vertex x="34.544" y="51.054"/>
+<vertex x="37.211" y="51.054"/>
+<vertex x="37.211" y="48.006"/>
+<vertex x="34.544" y="48.006"/>
 <vertex x="34.544" y="28.194"/>
 <vertex x="37.211" y="28.194"/>
@@
 </signal>
 <signal name="HDR_PWM6">
-<contactref element="TEENSY" pad="16/A2"/>
 <contactref element="FAN6" pad="1"/>
 <wire x1="21.1686875" y1="4.9794" x2="11.5306" y2="4.9794" width="0.1524" layer="16"/>
 <wire x1="8.89" y1="7.62" x2="11.5306" y2="4.9794" width="0.1524" layer="16"/>
-<wire x1="35.56" y1="34.258" x2="35.56" y2="34.29" width="0.1524" layer="16"/>
-<wire x1="22.7805" y1="6.5912125" x2="22.7805" y2="21.4785" width="0.1524" layer="16"/>
-<wire x1="22.7805" y1="6.5912125" x2="21.1686875" y2="4.9794" width="0.1524" layer="16"/>
-<wire x1="22.7805" y1="21.4785" x2="35.56" y2="34.258" width="0.1524" layer="16"/>
+<wire x1="21.1686875" y1="4.9794" x2="22.7805" y2="6.5912125" width="0.1524" layer="16"/>
+<contactref element="TEENSY" pad="22/A8"/>
+<wire x1="35.56" y1="49.53" x2="34.29" y2="48.26" width="0.1524" layer="16"/>
+<wire x1="34.29" y1="48.26" x2="32.54655" y2="48.26" width="0.1524" layer="16"/>
+<wire x1="32.54655" y1="48.26" x2="31.75" y2="47.46345" width="0.1524" layer="16"/>
+<wire x1="22.7805" y1="6.5912125" x2="31.75" y2="15.5607125" width="0.1524" layer="16"/>
+<wire x1="31.75" y1="15.5607125" x2="31.75" y2="47.46345" width="0.1524" layer="16"/>
 </signal>
 <signal name="HDR_PWM1">
@@
 <contactref element="R4" pad="1"/>
 <contactref element="R5" pad="1"/>
-<contactref element="JP1" pad="2"/>
 <contactref element="C2" pad="1"/>
 <wire x1="46.99" y1="12.065" x2="46.99" y2="13.97" width="0.635" layer="16"/>
 <contactref element="C3" pad="+"/>
-<wire x1="29.21" y1="43.18" x2="29.21" y2="48.26" width="0.508" layer="16"/>
-<wire x1="29.21" y1="48.26" x2="33.02" y2="52.07" width="0.508" layer="16"/>
-<wire x1="39.37" y1="43.18" x2="39.3446" y2="43.1546" width="0.508" layer="16"/>
-<wire x1="39.3446" y1="43.1546" x2="29.2354" y2="43.1546" width="0.508" layer="16"/>
-<wire x1="29.21" y1="43.18" x2="29.2354" y2="43.1546" width="0.508" layer="16"/>
 <wire x1="43.18" y1="17.78" x2="39.37" y2="17.78" width="0.508" layer="16"/>
 <wire x1="43.18" y1="17.78" x2="43.18" y2="15.24" width="0.508" layer="16"/>
@@
 <wire x1="43.18" y1="43.18" x2="44.69130625" y2="41.66869375" width="0.508" layer="16"/>
 <wire x1="44.69130625" y1="41.66869375" x2="44.69130625" y2="19.29130625" width="0.508" layer="16"/>
+<contactref element="SH1" pad="2"/>
+<wire x1="33.02" y1="52.07" x2="34.29" y2="50.8" width="0.508" layer="1"/>
+<wire x1="34.29" y1="50.8" x2="36.16045" y2="50.8" width="0.508" layer="1"/>
+<wire x1="36.16045" y1="50.8" x2="37.701725" y2="49.258725" width="0.508" layer="1"/>
+<wire x1="37.701725" y1="49.258725" x2="39.37" y2="47.59045" width="0.508" layer="1"/>
+<wire x1="39.37" y1="47.59045" x2="39.37" y2="43.18" width="0.508" layer="1"/>
+<wire x1="38.862" y1="50.546" x2="38.862" y2="50.419" width="0.508" layer="1"/>
+<wire x1="38.862" y1="50.419" x2="37.701725" y2="49.258725" width="0.508" layer="1"/>
 </signal>
 <signal name="V3.3" class="3">
 <contactref element="TEENSY" pad="3.3V3"/>
 <contactref element="TEENSY" pad="3.3V"/>
-<contactref element="JP1" pad="1"/>
-<wire x1="35.56" y1="54.61" x2="33.18920625" y2="54.61" width="0.508" layer="16"/>
-<wire x1="33.18920625" y1="54.61" x2="26.67" y2="48.09079375" width="0.508" layer="16"/>
-<wire x1="26.67" y1="48.09079375" x2="26.67" y2="43.18" width="0.508" layer="16"/>
-<wire x1="26.67" y1="43.18" x2="26.67" y2="30.48" width="0.508" layer="16"/>
-<wire x1="26.67" y1="30.48" x2="20.32" y2="24.13" width="0.508" layer="16"/>
+<contactref element="SH1" pad="1"/>
+<wire x1="29.972" y1="33.782" x2="20.32" y2="24.13" width="0.508" layer="16"/>
+<wire x1="29.972" y1="33.782" x2="29.972" y2="51.39279375" width="0.508" layer="16"/>
+<wire x1="29.972" y1="51.39279375" x2="33.18920625" y2="54.61" width="0.508" layer="16"/>
+<wire x1="33.18920625" y1="54.61" x2="35.56" y2="54.61" width="0.508" layer="16"/>
+<wire x1="35.56" y1="54.61" x2="36.068" y2="54.61" width="0.508" layer="1"/>
+<wire x1="38.862" y1="51.816" x2="36.068" y2="54.61" width="0.508" layer="1"/>
 </signal>
 </signals>
