File: Hardware/Simple/simple002/EAGLE/simple002.sch (EAGLE design)
At the start: 31 parts

Commit message: #8 hardware simple002 correct fan6 PWM to support Teensy 3.2, 3.5, 3.6, 4.0
Parts:
- removed JP1: JP1, jumper:JP1E
- added SH1: SHORTT5, shorts:SHORTT5
Connections:
- net AREF: now also SH1.P$2; no longer JP1.2
- net HDR_PWM6: now also TEENSY.22/A8/PWM; no longer TEENSY.16/A2
- net V3.3: now also SH1.P$1; no longer JP1.1
Other:
- note added: "Short to connect V3.3 to AREF"
- note removed: "Jumper to connect V3.3 to AREF (not used for Teensy 4.0)"
Changed lines of the file:
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@@
 <attribute name="MANUFACTURER_PART_NUMBER" value="C320C104M1U5TA7303"/>
-</part>
-<part name="JP1" library="jumper" library_urn="urn:adsk.eagle:library:252" deviceset="JP1E" device="" package3d_urn="urn:adsk.eagle:package:15455/1" value="JP1">
-<attribute name="DESC" value="Break Away Headers - Straight"/>
-<attribute name="DIGIKEY_PART_NUMBER" value="PRT-00116"/>
-<attribute name="MANUFACTURER" value="SparkFun Electronics"/>
-<attribute name="MANUFACTURER_PART_NUMBER" value="PRT-00116"/>
 </part>
 <part name="C1" library="capacitor-wima" library_urn="urn:adsk.eagle:library:116" deviceset="C" device="2,5-3" package3d_urn="urn:adsk.eagle:package:5436/1" value="0.1uF">
@@
 <attribute name="DESC" value="UNUSED"/>
 </part>
+<part name="SH1" library="shorts" deviceset="SHORT" device="T5"/>
 </parts>
 <sheets>
@@
 <text x="-78.74" y="109.22" size="1.778" layer="97">Header to connect GND to AGND
  (not needed in practice?)</text>
-<text x="-78.74" y="139.7" size="1.778" layer="97">Jumper to connect V3.3 to AREF
- (not used for Teensy 4.0)</text>
+<text x="-78.74" y="139.7" size="1.778" layer="97">Short to connect V3.3 to AREF</text>
 <text x="182.88" y="172.72" size="1.778" layer="97">Equivilent series resistors for thermistors
  (1% resistors, same resistance as thermistor nominal resistance)</text>
@@
 <attribute name="DESC" x="55.88" y="121.92" size="1.778" layer="96" display="off"/>
 </instance>
-<instance part="JP1" gate="A" x="-60.96" y="132.08" smashed="yes" rot="R270">
-<attribute name="NAME" x="-60.96" y="133.35" size="1.778" layer="95"/>
-<attribute name="VALUE" x="-60.96" y="126.365" size="1.778" layer="96"/>
-<attribute name="DIGIKEY_PART_NUMBER" x="-60.96" y="132.08" size="1.778" layer="96" rot="R270" display="off"/>
-<attribute name="DESC" x="-60.96" y="132.08" size="1.778" layer="96" rot="R270" display="off"/>
-<attribute name="MANUFACTURER" x="-60.96" y="132.08" size="1.778" layer="96" rot="R270" display="off"/>
-<attribute name="MANUFACTURER_PART_NUMBER" x="-60.96" y="132.08" size="1.778" layer="96" rot="R270" display="off"/>
-</instance>
 <instance part="C1" gate="G$1" x="45.72" y="121.92" smashed="yes">
 <attribute name="NAME" x="47.244" y="122.301" size="1.778" layer="95"/>
@@
 <attribute name="DESC" x="-58.42" y="101.6" size="1.778" layer="96" display="off"/>
 </instance>
+<instance part="SH1" gate="G$1" x="-58.42" y="132.08" smashed="yes">
+<attribute name="NAME" x="-60.6425" y="133.35" size="1.778" layer="95"/>
+</instance>
 </instances>
 <busses>
@@
 <net name="HDR_PWM6" class="0">
 <segment>
-<wire x1="-60.96" y1="226.06" x2="-78.74" y2="226.06" width="0.1524" layer="91"/>
-<pinref part="TEENSY" gate="G$1" pin="16/A2"/>
-<label x="-76.2" y="226.06" size="1.778" layer="95"/>
-</segment>
-<segment>
 <pinref part="FAN6" gate="G$1" pin="PWM"/>
 <wire x1="134.62" y1="236.22" x2="119.38" y2="236.22" width="0.1524" layer="91"/>
 <label x="121.92" y="236.22" size="1.778" layer="95"/>
 </segment>
+<segment>
+<pinref part="TEENSY" gate="G$1" pin="22/A8/PWM"/>
+<wire x1="-60.96" y1="210.82" x2="-78.74" y2="210.82" width="0.1524" layer="91"/>
+<label x="-76.2" y="210.82" size="1.778" layer="95"/>
+</segment>
 </net>
 <net name="HDR_PWM1" class="0">
@@
 </segment>
 <segment>
-<pinref part="JP1" gate="A" pin="2"/>
-<wire x1="-63.5" y1="129.54" x2="-76.2" y2="129.54" width="0.1524" layer="91"/>
-<label x="-73.66" y="129.54" size="1.778" layer="95"/>
-</segment>
-<segment>
 <pinref part="C2" gate="G$1" pin="1"/>
 <wire x1="101.6" y1="124.46" x2="101.6" y2="134.62" width="0.1524" layer="91"/>
@@
 <label x="116.84" y="127" size="1.778" layer="95" rot="R90"/>
 </segment>
+<segment>
+<pinref part="SH1" gate="G$1" pin="P$2"/>
+<wire x1="-55.88" y1="132.08" x2="-38.1" y2="132.08" width="0.1524" layer="91"/>
+<label x="-53.34" y="132.08" size="1.778" layer="95"/>
+</segment>
 </net>
 <net name="V3.3" class="3">
@@
 </segment>
 <segment>
-<pinref part="JP1" gate="A" pin="1"/>
-<wire x1="-63.5" y1="132.08" x2="-76.2" y2="132.08" width="0.1524" layer="91"/>
+<pinref part="SH1" gate="G$1" pin="P$1"/>
+<wire x1="-60.96" y1="132.08" x2="-76.2" y2="132.08" width="0.1524" layer="91"/>
 <label x="-73.66" y="132.08" size="1.778" layer="95"/>
 </segment>
